File: model-railroad-electric-conection-coupler/male/male.kicad_sch (KiCad schematic)
At the start: 3 parts, among them J1 Conn_01x03_Pin, J2 Conn_01x06_Pin, J3 Conn_01x03_Pin

Commit message: 鉄道模型用の通電カプラー PCB 版 WIP
Parts:
- J1, J3: footprint (none) -> Library:Pin_Side
- J2: footprint (none) -> Connector_Molex:Molex_PicoBlade_53048-0610_1x06_P1.25mm_Horizontal
Connections:
- net at J2.1 (Pin_1): now also J1.3 (Pin_3); no longer J1.1 (Pin_1)
- net at J2.3 (Pin_3): now also J1.1 (Pin_1); no longer J1.3 (Pin_3)
Changed lines of the file:
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@@
+	(wire
+		(pts
+			(xy 125.73 86.36) (xy 125.73 106.68)
+		)
+		(stroke
+			(width 0)
+			(type default)
+		)
+	)
+	(wire
+		(pts
+			(xy 80.01 73.66) (xy 85.09 73.66)
+		)
+		(stroke
+			(width 0)
+			(type default)
+		)
+	)
+	(wire
+		(pts
+			(xy 80.01 68.58) (xy 90.17 68.58)
+		)
+		(stroke
+			(width 0)
+			(type default)
+		)
+	)
 	(wire
 		(pts
@@
 	(wire
 		(pts
-			(xy 125.73 86.36) (xy 125.73 106.68)
-		)
-		(stroke
-			(width 0)
-			(type default)
-		)
-	)
-	(wire
-		(pts
 			(xy 128.27 109.22) (xy 59.69 109.22)
 		)
@@
 	(wire
 		(pts
-			(xy 90.17 73.66) (xy 90.17 101.6)
-		)
-		(stroke
-			(width 0)
-			(type default)
-		)
-	)
-	(wire
-		(pts
-			(xy 80.01 68.58) (xy 85.09 68.58)
+			(xy 90.17 68.58) (xy 90.17 101.6)
 		)
 		(stroke
@@
 	(wire
 		(pts
-			(xy 80.01 73.66) (xy 90.17 73.66)
-		)
-		(stroke
-			(width 0)
-			(type default)
-		)
-	)
-	(wire
-		(pts
 			(xy 119.38 88.9) (xy 128.27 88.9)
 		)
@@
 	(wire
 		(pts
-			(xy 85.09 68.58) (xy 85.09 96.52)
+			(xy 85.09 73.66) (xy 85.09 96.52)
 		)
 		(stroke
@@
 			)
 		)
-		(property "Footprint" ""
+		(property "Footprint" "Library:Pin_Side"
 			(at 114.3 86.36 0)
 			(hide yes)
@@
 			)
 		)
-		(property "Footprint" ""
+		(property "Footprint" "Connector_Molex:Molex_PicoBlade_53048-0610_1x06_P1.25mm_Horizontal"
 			(at 54.61 101.6 0)
 			(hide yes)
@@
 			)
 		)
-		(property "Footprint" ""
+		(property "Footprint" "Library:Pin_Side"
 			(at 74.93 71.12 0)
 			(hide yes)
