File: model-railroad-electric-conection-coupler/pcb/coupler.kicad_pcb (KiCad board)
At the start: 2 copper layers, 10 x 27.2 mm, 5 parts, among them J1 Conn_01x03_Pin, J2 Conn_01x06_Pin, J3 Conn_01x03_Pin

Commit message: [model-railroad-electric-conection-coupler] 連結端子のパッドを大きく はんだ付けしやすく
Parts:
- moved J1 0.10 mm to (35.0, 31.9)
- moved J3 0.10 mm to (35.0, 31.9)
Changed lines of the file:
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@@
 	(footprint "Library:Pin_Side"
 		(layer "F.Cu")
-		(at 34.99 31.79 -90)
+		(at 34.99 31.89 -90)
 		(property "Reference" "J3"
 			(at 2.71 -0.01 0)
@@
 		(pad "1" smd roundrect
 			(at 0 1.27 270)
-			(size 2.54 0.4)
+			(size 3 0.6)
 			(layers "*.Mask" "B.Cu")
 			(roundrect_rratio 0.15)
@@
 		(pad "2" smd roundrect
 			(at 0 0 270)
-			(size 2.54 0.4)
+			(size 3 0.6)
 			(layers "*.Mask" "B.Cu")
 			(roundrect_rratio 0.15)
@@
 		(pad "3" smd roundrect
 			(at 0 -1.27 270)
-			(size 2.54 0.4)
+			(size 3 0.6)
 			(layers "*.Mask" "B.Cu")
 			(roundrect_rratio 0.15)
@@
 	(footprint "Library:Pin_Side"
 		(layer "B.Cu")
-		(at 34.99 31.79 90)
+		(at 34.99 31.89 90)
 		(property "Reference" "J1"
 			(at -2.71 0.01 0)
@@
 		(pad "1" smd roundrect
 			(at 0 -1.27 90)
-			(size 2.54 0.4)
+			(size 3 0.6)
 			(layers "*.Mask" "F.Cu")
 			(roundrect_rratio 0.15)
@@
 		(pad "2" smd roundrect
 			(at 0 0 90)
-			(size 2.54 0.4)
+			(size 3 0.6)
 			(layers "*.Mask" "F.Cu")
 			(roundrect_rratio 0.15)
@@
 		(pad "3" smd roundrect
 			(at 0 1.27 90)
-			(size 2.54 0.4)
+			(size 3 0.6)
 			(layers "*.Mask" "F.Cu")
 			(roundrect_rratio 0.15)
@@
 	)
 	(segment
-		(start 33.72 31.79)
-		(end 33.72 34.860202)
-		(width 0.2)
-		(layer "B.Cu")
-		(net "Net-(J2-Pin_4)")
-	)
-	(segment
 		(start 35.639949 44.7)
 		(end 35.65 44.7)
@@
 	)
 	(segment
+		(start 33.72 34.860202)
+		(end 33.72 31.89)
+		(width 0.2)
+		(layer "B.Cu")
+		(net "Net-(J2-Pin_4)")
+	)
+	(segment
 		(start 33.72 31.79)
 		(end 33.723838 31.793838)
@@
 	(segment
 		(start 34.99 35.564516)
-		(end 34.99 31.79)
+		(end 34.99 31.89)
 		(width 0.2)
 		(layer "B.Cu")
@@
 	)
 	(segment
+		(start 38.6 38.608831)
+		(end 36.26 36.26883)
+		(width 0.2)
+		(layer "B.Cu")
+		(net "Net-(J2-Pin_6)")
+	)
+	(segment
+		(start 38.6 41.631372)
+		(end 38.6 38.608831)
+		(width 0.2)
+		(layer "B.Cu")
+		(net "Net-(J2-Pin_6)")
+	)
+	(segment
 		(start 38.15 42.081372)
-		(end 38.15 44.7)
+		(end 38.6 41.631372)
 		(width 0.2)
 		(layer "B.Cu")
@@
 	)
 	(segment
-		(start 38.6 38.608831)
-		(end 38.6 41.631372)
+		(start 36.26 36.26883)
+		(end 36.26 31.89)
 		(width 0.2)
 		(layer "B.Cu")
@@
 	)
 	(segment
-		(start 36.26 36.26883)
-		(end 38.6 38.608831)
-		(width 0.2)
-		(layer "B.Cu")
-		(net "Net-(J2-Pin_6)")
-	)
-	(segment
-		(start 36.26 31.79)
-		(end 36.26 36.26883)
+		(start 38.15 44.7)
+		(end 38.15 42.081372)
 		(width 0.2)
 		(layer "B.Cu")
@@
 	)
 	(segment
-		(start 38.6 41.631372)
-		(end 38.15 42.081372)
-		(width 0.2)
-		(layer "B.Cu")
-		(net "Net-(J2-Pin_6)")
-	)
-	(segment
 		(start 38.2 44.65)
 		(end 38.15 44.7)
@@
 	)
 	(segment
-		(start 33.72 31.79)
-		(end 33.72 33.664313)
+		(start 33.72 33.664313)
+		(end 33.72 31.89)
 		(width 0.2)
 		(layer "F.Cu")
@@
 	)
 	(segment
-		(start 34.99 32.959999)
-		(end 32.2 35.749999)
+		(start 34.99 32.959998)
+		(end 34.874999 33.074999)
 		(width 0.2)
 		(layer "F.Cu")
@@
 	)
 	(segment
+		(start 34.99 31.89)
+		(end 34.99 32.959998)
+		(width 0.2)
+		(layer "F.Cu")
+		(net "Net-(J1-Pin_2)")
+	)
+	(segment
+		(start 34.874999 33.074999)
+		(end 32.2 35.749999)
+		(width 0.2)
+		(layer "F.Cu")
+		(net "Net-(J1-Pin_2)")
+	)
+	(segment
+		(start 34.99 32.959999)
+		(end 34.874999 33.074999)
+		(width 0.2)
+		(layer "F.Cu")
+		(net "Net-(J1-Pin_2)")
+	)
+	(segment
 		(start 32.2 43.5)
 		(end 33.15 44.45)
@@
 		(width 0.2)
 		(layer "F.Cu")
-		(net "Net-(J1-Pin_2)")
-	)
-	(segment
-		(start 34.99 31.79)
-		(end 34.99 32.959999)
-		(width 0.2)
-		(layer "F.Cu")
